File: circuit/determOfchromiumOxideDevice.kicad_pcb (KiCad board)
At the start: 2 copper layers, 60.3 x 95.2 mm, 61 parts, among them IC1 ATTINY2313-P, IC2 ATMEGA8A-A, K1 CONN_INPUT_OPTO_INT, P1 CONN_SENSOR_LED_POW, P2 CONN_SENSOR_SIGNAL_IN, P3 CONN_USB, P4 CONN_ISP, P5 CONN_POWER, P6 CONN_BTN_START_STOP, P7 CONN_OUT_IND_PROC_LED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

Commit message: На схеме: добавлено описание какой Ку нужно установить, изменены номиналы R для ОУ, изменен номинал С3. Исправлена ошибка монтажа - были перепутаны usb data которые идут на tn2313, D+ был не туда подключен. МК теперь подключен к питанию 3,3 В. Внесены соотв. изменения в pcb.
Parts:
- added D8: LED-Y, LED-5MM, F.Cu at (59.1, 185.4)
- C3: value 0.1uF -> 0.01uF
- R1: value 5.1k -> 910
- RV2: value 68k -> 33k
- moved R3 16.5 mm to (64.8, 141.0), turned to 0 degrees
- moved R4 1.91 mm to (72.4, 157.5)
Connections:
- C5 pad 1: VCC -> +3.3V
- IC1 pad 20: VCC -> +3.3V
- IC1 pad 6: (no net) -> /USB_D+
- IC1 pad 8: /USB_D+ -> (no net)
- R2 pad 2: VCC -> +3.3V
- R3 pad 2: VCC -> +3.3V
Routing:
- net +3.3V: track 0.00 -> 74.7 mm, vias 0 -> 1
- net VCC: track 405.3 -> 373.7 mm, vias 12 -> 10
- net GND: track 466.6 -> 485.4 mm, vias 6 -> 8
- net /USB_D+: track 4.13 -> 8.28 mm, vias 0 -> 2
- net /USB_D-: track 4.13 -> 6.35 mm
- net N-0000027: track 27.5 -> 29.1 mm
