File: circuit/determOfchromiumOxideDevice.sch (KiCad schematic (older format))
At the start: 61 parts, among them IC1 ATTINY2313-P, IC2 ATMEGA8A-A, K1 CONN_INPUT_OPTO_INT, P1 CONN_SENSOR_LED_POW, P2 CONN_SENSOR_SIGNAL_IN, P3 CONN_USB, P4 CONN_ISP, P5 CONN_POWER, P6 CONN_BTN_START_STOP, P7 CONN_OUT_IND_PROC_LED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

Commit message: На схеме: добавлено описание какой Ку нужно установить, изменены номиналы R для ОУ, изменен номинал С3. Исправлена ошибка монтажа - были перепутаны usb data которые идут на tn2313, D+ был не туда подключен. МК теперь подключен к питанию 3,3 В. Внесены соотв. изменения в pcb.
Parts:
- added D8: LED-Y, ~, symbol LED
- C3: value 0.1uF -> 0.01uF
- R1: value 5.1k -> 910
- RV2: value 68k -> 33k
Connections:
- net labels added: +3,3V
- wire segments 107 -> 111
Other:
- note added: "Kу подстр = 1+(22/0,910)=25,17"
- note added: "Uin = 100mV; Uout = 100mV*25~2.56V"
- note added: "Zener diode do not used !!! \nInsted of them tn2313 connected to supply +3.3V ."
- note added: "usb mcu\n------------\nD+ int0 PD2\nD- int1 PD3"
Changed lines of the file:
@@
 Sheet 1 1
 Title ""
-Date "31 oct 2015"
+Date "10 dec 2015"
 Rev ""
 Comp ""
@@
 P 2825 1650
 F 0 "RV2" H 2825 1550 39  0000 C CNN
-F 1 "68k" H 2825 1650 39  0000 C CNN
+F 1 "33k" H 2825 1650 39  0000 C CNN
 F 2 "~" H 2825 1650 60  0000 C CNN
 F 3 "~" H 2825 1650 60  0000 C CNN
@@
 P 1425 1950
 F 0 "R1" V 1505 1950 40  0000 C CNN
-F 1 "5.1k" V 1432 1951 40  0000 C CNN
+F 1 "910" V 1432 1951 40  0000 C CNN
 F 2 "~" V 1355 1950 30  0000 C CNN
 F 3 "~" H 1425 1950 30  0000 C CNN
@@
 P 1550 1500
 F 0 "C3" H 1550 1600 40  0000 L CNN
-F 1 "0.1uF" H 1556 1415 40  0000 L CNN
+F 1 "0.01uF" H 1556 1415 40  0000 L CNN
 F 2 "~" H 1588 1350 30  0000 C CNN
 F 3 "~" H 1550 1500 60  0000 C CNN
@@
 L VCC #PWR020
 U 1 1 56347D14
-P 2225 3200
-F 0 "#PWR020" H 2225 3300 30  0001 C CNN
-F 1 "VCC" H 2225 3300 30  0000 C CNN
-F 2 "" H 2225 3200 60  0000 C CNN
-F 3 "" H 2225 3200 60  0000 C CNN
-	1    2225 3200
+P 2975 3300
+F 0 "#PWR020" H 2975 3400 30  0001 C CNN
+F 1 "VCC" H 2975 3400 30  0000 C CNN
+F 2 "" H 2975 3300 60  0000 C CNN
+F 3 "" H 2975 3300 60  0000 C CNN
+	1    2975 3300
 	1    0    0    -1
 $EndComp
@@
 	-1   0    0    1
 $EndComp
-$Comp
-L ZENERSMALL D1
-U 1 1 56347E59
-P 1875 4125
-F 0 "D1" H 1825 4225 40  0000 C CNN
-F 1 "3V6" H 1925 4225 30  0000 C CNN
-F 2 "~" H 1875 4125 60  0000 C CNN
-F 3 "~" H 1875 4125 60  0000 C CNN
-	1    1875 4125
-	0    -1   -1   0
-$EndComp
-$Comp
-L ZENERSMALL D2
-U 1 1 56347E83
-P 2075 4125
-F 0 "D2" H 2025 4225 40  0000 C CNN
-F 1 "3V6" H 2125 4225 30  0000 C CNN
-F 2 "~" H 2075 4125 60  0000 C CNN
-F 3 "~" H 2075 4125 60  0000 C CNN
-	1    2075 4125
-	0    -1   -1   0
-$EndComp
 Text Label 2825 3950 0    39   ~ 0
 USB_D+
@@
 F 3 "" H 2575 6275 60  0000 C CNN
 	1    2575 6275
-	1    0    0    -1
-$EndComp
-$Comp
-L VCC #PWR021
-U 1 1 5634868F
-P 2575 4900
-F 0 "#PWR021" H 2575 5000 30  0001 C CNN
-F 1 "VCC" H 2575 5000 30  0000 C CNN
-F 2 "" H 2575 4900 60  0000 C CNN
-F 3 "" H 2575 4900 60  0000 C CNN
-	1    2575 4900
 	1    0    0    -1
 $EndComp
@@
 $EndComp
 $Comp
-L GND #PWR022
+L GND #PWR021
 U 1 1 563486A1
 P 3025 5150
-F 0 "#PWR022" H 3025 5150 30  0001 C CNN
+F 0 "#PWR021" H 3025 5150 30  0001 C CNN
 F 1 "GND" H 3025 5080 30  0001 C CNN
 F 2 "" H 3025 5150 60  0000 C CNN
@@
 $EndComp
 $Comp
-L GND #PWR023
+L GND #PWR022
 U 1 1 563486B9
 P 650 6325
-F 0 "#PWR023" H 650 6325 30  0001 C CNN
+F 0 "#PWR022" H 650 6325 30  0001 C CNN
 F 1 "GND" H 650 6255 30  0001 C CNN
 F 2 "" H 650 6325 60  0000 C CNN
@@
 Text Label 3725 6675 0    39   ~ 0
 USB_D-
-Text Label 3725 6775 0    39   ~ 0
+Text Label 3725 6575 0    39   ~ 0
 USB_D+
 NoConn ~ 3725 6975
 NoConn ~ 3725 6875
-NoConn ~ 3725 6575
 NoConn ~ 3725 6175
 NoConn ~ 3725 6075
@@
 $EndComp
 $Comp
-L GND #PWR024
+L GND #PWR023
 U 1 1 563495F4
 P 6125 5525
-F 0 "#PWR024" H 6125 5525 30  0001 C CNN
+F 0 "#PWR023" H 6125 5525 30  0001 C CNN
 F 1 "GND" H 6125 5455 30  0001 C CNN
 F 2 "" H 6125 5525 60  0000 C CNN
@@
 $EndComp
 $Comp
-L VCC #PWR025
+L VCC #PWR024
 U 1 1 563495FA
 P 5525 2200
-F 0 "#PWR025" H 5525 2300 30  0001 C CNN
+F 0 "#PWR024" H 5525 2300 30  0001 C CNN
 F 1 "VCC" H 5525 2300 30  0000 C CNN
 F 2 "" H 5525 2200 60  0000 C CNN
@@
 $EndComp
 $Comp
-L GND #PWR026
+L GND #PWR025
 U 1 1 56349606
 P 6600 2475
-F 0 "#PWR026" H 6600 2475 30  0001 C CNN
+F 0 "#PWR025" H 6600 2475 30  0001 C CNN
 F 1 "GND" H 6600 2405 30  0001 C CNN
 F 2 "" H 6600 2475 60  0000 C CNN
@@
 $EndComp
 $Comp
-L GND #PWR027
+L GND #PWR026
 U 1 1 56349624
 P 4500 4300
-F 0 "#PWR027" H 4500 4300 30  0001 C CNN
+F 0 "#PWR026" H 4500 4300 30  0001 C CNN
 F 1 "GND" H 4500 4230 30  0001 C CNN
 F 2 "" H 4500 4300 60  0000 C CNN
@@
 res
 $Comp
-L VCC #PWR028
+L VCC #PWR027
 U 1 1 5634A75F
 P 6575 1250
-F 0 "#PWR028" H 6575 1350 30  0001 C CNN
+F 0 "#PWR027" H 6575 1350 30  0001 C CNN
 F 1 "VCC" H 6575 1350 30  0000 C CNN
 F 2 "" H 6575 1250 60  0000 C CNN
@@
 $EndComp
 $Comp
-L GND #PWR029
+L GND #PWR028
 U 1 1 5634A76B
 P 6575 1500
-F 0 "#PWR029" H 6575 1500 30  0001 C CNN
+F 0 "#PWR028" H 6575 1500 30  0001 C CNN
 F 1 "GND" H 6575 1430 30  0001 C CNN
 F 2 "" H 6575 1500 60  0000 C CNN
@@
 	1875 4025 1875 3875
 Connection ~ 1875 3875
-Wire Wire Line
-	2075 4025 2075 3775
 Connection ~ 2075 3775
 Wire Wire Line
@@
 NoConn ~ 1625 3675
 $Comp
-L GND #PWR030
+L GND #PWR029
 U 1 1 56348689
 P 2575 7325
-F 0 "#PWR030" H 2575 7325 30  0001 C CNN
+F 0 "#PWR029" H 2575 7325 30  0001 C CNN
 F 1 "GND" H 2575 7255 30  0001 C CNN
 F 2 "" H 2575 7325 60  0000 C CNN
@@
 Connection ~ 3700 1650
 Connection ~ 3500 1400
+Text Notes 2300 2100 0    39   ~ 0
+Kу подстр = 1+(22/0,910)=25,17
+Text Notes 2300 2200 0    39   ~ 0
+Uin = 100mV; Uout = 100mV*25~2.56V
+Text Notes 1750 4350 0    39   ~ 0
+Zener diode do not used !!! \nInsted of them tn2313 connected to supply +3.3V .
+NoConn ~ 3725 6775
+Text Notes 3900 5650 0    39   ~ 0
+usb    mcu\n------------\nD+      int0 PD2\nD-       int1 PD3
+$Comp
+L LED D8
+U 1 1 5669BBA7
+P 3275 3400
+F 0 "D8" H 3275 3500 50  0000 C CNN
+F 1 "LED-Y" H 3275 3300 50  0000 C CNN
+F 2 "~" H 3275 3400 60  0000 C CNN
+F 3 "~" H 3275 3400 60  0000 C CNN
+	1    3275 3400
+	1    0    0    -1
+$EndComp
+$Comp
+L +3,3V #PWR030
+U 1 1 5669BBC0
+P 3625 3300
+F 0 "#PWR030" H 3625 3260 30  0001 C CNN
+F 1 "+3,3V" H 3625 3410 30  0000 C CNN
+F 2 "" H 3625 3300 60  0000 C CNN
+F 3 "" H 3625 3300 60  0000 C CNN
+	1    3625 3300
+	1    0    0    -1
+$EndComp
+Wire Wire Line
+	3075 3400 2975 3400
+Wire Wire Line
+	2975 3400 2975 3300
+Wire Wire Line
+	3475 3400 3625 3400
+Wire Wire Line
+	3625 3400 3625 3300
+$Comp
+L +3,3V #PWR031
+U 1 1 5669BD3B
+P 2225 3200
+F 0 "#PWR031" H 2225 3160 30  0001 C CNN
+F 1 "+3,3V" H 2225 3310 30  0000 C CNN
+F 2 "" H 2225 3200 60  0000 C CNN
+F 3 "" H 2225 3200 60  0000 C CNN
+	1    2225 3200
+	1    0    0    -1
+$EndComp
+$Comp
+L +3,3V #PWR032
+U 1 1 5669BD41
+P 2575 4900
+F 0 "#PWR032" H 2575 4860 30  0001 C CNN
+F 1 "+3,3V" H 2575 5010 30  0000 C CNN
+F 2 "" H 2575 4900 60  0000 C CNN
+F 3 "" H 2575 4900 60  0000 C CNN
+	1    2575 4900
+	1    0    0    -1
+$EndComp
+Wire Wire Line
+	2075 4025 2075 3775
+$Comp
+L ZENERSMALL D2
+U 1 1 56347E83
+P 2075 4125
+F 0 "D2" H 2025 4225 40  0000 C CNN
+F 1 "3V6" H 2125 4225 30  0000 C CNN
+F 2 "~" H 2075 4125 60  0000 C CNN
+F 3 "~" H 2075 4125 60  0000 C CNN
+	1    2075 4125
+	0    -1   -1   0
+$EndComp
+$Comp
+L ZENERSMALL D1
+U 1 1 56347E59
+P 1875 4125
+F 0 "D1" H 1825 4225 40  0000 C CNN
+F 1 "3V6" H 1925 4225 30  0000 C CNN
+F 2 "~" H 1875 4125 60  0000 C CNN
+F 3 "~" H 1875 4125 60  0000 C CNN
+	1    1875 4125
+	0    -1   -1   0
+$EndComp
 $EndSCHEMATC

Commit message: Modified circuit and export to png.
Other:
- note added: "Uin = 100mV; Uout = 100mV*25=2.56V"
- note removed: "Uin = 100mV; Uout = 100mV*25~2.56V"
Changed lines of the file:
@@
 Kу подстр = 1+(22/0,910)=25,17
 Text Notes 2300 2200 0    39   ~ 0
-Uin = 100mV; Uout = 100mV*25~2.56V
+Uin = 100mV; Uout = 100mV*25=2.56V
 Text Notes 1750 4350 0    39   ~ 0
 Zener diode do not used !!! \nInsted of them tn2313 connected to supply +3.3V .

Commit message: Changed input photo signal part in schematic - added RV and emitter repeater cascade in LM324. Changed amp gain.Important - input part in LM324 in schematic do not match from PCB layout.
Parts:
- added RV4: 10k, ~, symbol POT
- added RV5: 100k, ~, symbol POT
- added unit 1 of U1
- C3: value 0.01uF -> 10uF
- R1: value 910 -> 35k
- RV2: value 33k -> 200k
Connections:
- wire segments 111 -> 127
Other:
- note removed: "Kу подстр = 1+(22/0,910)=25,17"
- note removed: "Uin = 100mV; Uout = 100mV*25=2.56V"
- moved on the sheet: C3, C4, P1, P2, R1, R6, RV1, RV2, RV3
