File: circuit/powerUnit.sch (KiCad schematic (older format))
At the start: 34 parts, among them M1 Stepper_Motor_unipolar_5pin, Q1 IRLML0030, Q2 IRLML0030, Q3 IRLML0030, Q4 IRLML0030, U6 MP1584EN-LF-Z

Commit message: In powerUnit.sch changed 15uHn to 15uH.
Parts:
- L4: value 15uHn -> 15uH
Changed lines of the file:
@@
 AR Path="/5BCAEDBB/5BCDDCA3" Ref="L4"  Part="1"
 F 0 "L4" V 5025 3500 50  0000 C CNN
-F 1 "15uHn" V 5025 3275 50  0000 C CNN
+F 1 "15uH" V 5025 3275 50  0000 C CNN
 F 2 "Inductor_SMD:L_12x12mm_H6mm" H 4950 3350 50  0001 C CNN
 F 3 "~" H 4950 3350 50  0001 C CNN

Commit message: Added articles for some components in powerUnit schematic.
Parts:
- C31: Article - -> 000013353
- RV5: Article - -> 000012071
- U6: symbol MP1584EN-LF-Z:MP1584EN-LF-Z -> surfaceActivationScanner-rescue:MP1584EN-LF-Z-MP1584EN-LF-Z; Article (none) -> 000011495
Changed lines of the file:
@@
 $EndComp
 $Comp
-L MP1584EN-LF-Z:MP1584EN-LF-Z U?
+L surfaceActivationScanner-rescue:MP1584EN-LF-Z-MP1584EN-LF-Z U?
 U 1 1 5BCDDC77
 P 3600 3650
@@
 F 4 "Monolithic Power" H 3600 3650 50  0001 L BNN "Field4"
 F 5 "SOIC-8 Monolithic Power Systems" H 3600 3650 50  0001 L BNN "Field5"
+F 6 "000011495" H 3600 3650 50  0001 C CNN "Article"
 	1    3600 3650
 	1    0    0    -1
@@
 F 2 "Potentiometer_THT:Potentiometer_Vishay_T7-YA_Single_Vertical" H 5450 4050 50  0001 C CNN
 F 3 "~" H 5450 4050 50  0001 C CNN
-F 4 "-" V 5450 4050 50  0001 C CNN "Article"
+F 4 "000012071" V 5450 4050 50  0001 C CNN "Article"
 	1    5450 4050
 	0    -1   -1   0
@@
 F 2 "Capacitor_SMD:C_0805_2012Metric" H 4463 4050 50  0001 C CNN
 F 3 "~" H 4425 4200 50  0001 C CNN
-F 4 "-" H 4425 4200 50  0001 C CNN "Article"
+F 4 "000013353" H 4425 4200 50  0001 C CNN "Article"
 	1    4425 4200
 	1    0    0    -1
