File: circuit/surfaceActivationScanner.sch (KiCad schematic (older format))
At the start: 64 parts, among them J1 Conn_power, J2 Conn_sensor_led, J3 Conn_opto_int, J4 Conn_sensor_VT, J5 Conn btn start/stop msr, J6 Conn led start/stop msr, J7 Conn_USB, J8 AVR-ISP-6, U1 AP1117-50, U2 MCP3421A0T-ECH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

Commit message: Fix bug in schematic - added connection SM enable from DC-DC convertor to MCU.
Parts:
- U4: footprint (none) -> Package_SO:SOIC-14_3.9x8.7mm_P1.27mm
Connections:
- wire segments 215 -> 216
- no-connect marks 20 -> 19
Changed lines of the file:
@@
 F 0 "U4" H 2700 4267 50  0000 C CNN
 F 1 "LM324" H 2700 4176 50  0000 C CNN
-F 2 "" H 2650 4000 50  0001 C CNN
+F 2 "Package_SO:SOIC-14_3.9x8.7mm_P1.27mm" H 2650 4000 50  0001 C CNN
 F 3 "http://www.ti.com/lit/ds/symlink/lm2902-n.pdf" H 2750 4100 50  0001 C CNN
 F 4 "000000020" H 2700 3900 50  0001 C CNN "Article"
@@
 NoConn ~ 7300 3825
 NoConn ~ 7300 3925
-NoConn ~ 7300 4425
 NoConn ~ 1400 7050
 NoConn ~ 1400 6850
@@
 Wire Wire Line
 	4025 1375 4275 1375
+Wire Wire Line
+	7900 4425 7300 4425
 Wire Bus Line
 	5075 5675 8000 5675
@@
 Wire Bus Line
 	8000 2500 8000 5675
+Entry Wire Line
+	7900 4425 8000 4525
+Text Label 7875 4425 2    50   ~ 0
+smen
 $EndSCHEMATC

Commit message: Added articles for some components in main schematic.
Parts:
- C3: Article - -> 000006671
- RV1: Article (none) -> 000012071
- U3: symbol MCU_Microchip_ATmega:ATmega8-16AU -> surfaceActivationScanner-rescue:ATmega8-16AU-MCU_Microchip_ATmega
- U5: Article - -> 000002281
- Y1: Article - -> 000003646
Changed lines of the file:
@@
 $EndDescr
 $Comp
-L MCU_Microchip_ATmega:ATmega8-16AU U3
+L surfaceActivationScanner-rescue:ATmega8-16AU-MCU_Microchip_ATmega U3
 U 1 1 5BC410A9
 P 6700 3725
@@
 F 2 "Package_SO:SSOP-28_5.3x10.2mm_P0.65mm" H 2200 6650 50  0001 C CNN
 F 3 "http://www.ftdichip.com/Products/ICs/FT232RL.htm" H 2200 6650 50  0001 C CNN
-F 4 "-" H 2200 6650 50  0001 C CNN "Article"
+F 4 "000002281" H 2200 6650 50  0001 C CNN "Article"
 	1    2200 6650
 	1    0    0    -1
@@
 F 2 "Potentiometer_THT:Potentiometer_Vishay_T7-YA_Single_Vertical" H 1550 2650 50  0001 C CNN
 F 3 "~" H 1550 2650 50  0001 C CNN
+F 4 "000012071" V 1550 2650 50  0001 C CNN "Article"
 	1    1550 2650
 	0    -1   -1   0
@@
 F 2 "Crystal:Crystal_HC49-U_Vertical" H 6000 2825 50  0001 C CNN
 F 3 "~" H 6000 2825 50  0001 C CNN
-F 4 "-" V 6000 2825 50  0001 C CNN "Article"
+F 4 "000003646" V 6000 2825 50  0001 C CNN "Article"
 	1    6000 2825
 	0    -1   -1   0
@@
 F 2 "Capacitor_Tantalum_SMD:CP_EIA-3528-21_Kemet-B" H 4275 1175 50  0001 C CNN
 F 3 "~" H 4275 1175 50  0001 C CNN
-F 4 "-" H 4275 1175 50  0001 C CNN "Article"
+F 4 "000006671" H 4275 1175 50  0001 C CNN "Article"
 	1    4275 1175
 	1    0    0    -1
@@
 Wire Wire Line
 	7900 4425 7300 4425
+Entry Wire Line
+	7900 4425 8000 4525
+Text Label 7875 4425 2    50   ~ 0
+smen
 Wire Bus Line
 	5075 5675 8000 5675
@@
 Wire Bus Line
 	8000 2500 8000 5675
-Entry Wire Line
-	7900 4425 8000 4525
-Text Label 7875 4425 2    50   ~ 0
-smen
 $EndSCHEMATC
